File: pcb_design_kicad/ats.kicad_sch (KiCad schematic)
At the start: 37 parts, among them J1 Screw_Terminal_01x03, J2 Conn_01x12_Female, J3 Screw_Terminal_01x03, J4 Screw_Terminal_01x02, J6 Screw_Terminal_01x02, K1 FINDER-32.21-x300, K2 FINDER-32.21-x300, Q1 BC547, Q2 BC547, U1 LM7805_TO220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

Commit message: update pcb
Parts:
- removed J2: Conn_01x12_Female, Connector_PinHeader_2.54mm:PinHeader_1x12_P2.54mm_Vertical, symbol Connector:Conn_01x12_Female
- added C3: 2200u, Capacitor_THT:C_Radial_D10.0mm_H12.5mm_P5.00mm, symbol Device:C
- added D12, D3, D4, D5, D6: 1N4007, Diode_THT:D_DO-41_SOD81_P10.16mm_Horizontal, symbol Diode:1N4007
- added D8: LED, LED_THT:LED_D3.0mm, symbol Device:LED
- added J2: Screw_Terminal_01x03, TerminalBlock_Phoenix:TerminalBlock_Phoenix_MKDS-3-3-5.08_1x03_P5.08mm_Horizontal, symbol Connector:Screw_Terminal_01x03
- added J7, J8: Screw_Terminal_01x02, TerminalBlock_Phoenix:TerminalBlock_Phoenix_MKDS-1,5-2-5.08_1x02_P5.08mm_Horizontal, symbol Connector:Screw_Terminal_01x02
- added K3: FINDER-32.21-x300, Relay_THT:Relay_SPDT_Finder_36.11, symbol Relay:FINDER-32.21-x300
- added Q3: BC547, Package_TO_SOT_THT:TO-92_Inline, symbol Transistor_BJT:BC547
- added R11: 330, Resistor_THT:R_Axial_DIN0204_L3.6mm_D1.6mm_P7.62mm_Horizontal, symbol Device:R
- added R15, R4: 10k, Resistor_THT:R_Axial_DIN0204_L3.6mm_D1.6mm_P7.62mm_Horizontal, symbol Device:R
- added R3: 100k, Resistor_THT:R_Axial_DIN0204_L3.6mm_D1.6mm_P7.62mm_Horizontal, symbol Device:R
- added R8: 1k, Resistor_THT:R_Axial_DIN0204_L3.6mm_D1.6mm_P7.62mm_Horizontal, symbol Device:R
- added U3: LM7805_TO220, Package_TO_SOT_THT:TO-220-3_Vertical, symbol Regulator_Linear:LM7805_TO220
- added U6: LCD-016N002L, Display:LCD-016N002L, symbol Display_Character:LCD-016N002L
Connections:
- net +12V: now also D12.1 (K), K3.A1
- net +5V: now also U6.2 (VDD), U6.5 (R/~{W})
- net 7: now also R15.1; no longer R14.1
- net D4: now also U6.11 (DB4)
- net D5: now also U6.12 (DB5)
- net D6: now also U6.13 (DB6)
- net D7: now also U6.14 (DB7)
- net E: now also U6.6 (E)
- net GND: now also C3.2, D8.1 (K), J2.1 (Pin_1), Q3.3 (E), R4.2, R8.2, U3.2 (GND), U6.1 (VSS); no longer J3.2 (Pin_2), J6.1 (Pin_1)
- net PIN11: now also J7.2 (Pin_2), J8.2 (Pin_2), K3.11
- net RL1: now also J6.1 (Pin_1); no longer C2.1, D1.1 (K), D2.1 (K), R1.1, R7.1, U2.1 (VI)
- net RL2: now also J7.1 (Pin_1); no longer C4.1, J3.3 (Pin_3), R5.1, R9.1, U4.1 (VI)
- net RS: now also U6.4 (RS)
- net VEE: now also U6.15 (A/VEE)
- net 6: now reaches U5.13 (PD7)
- net 6: now also R14.1
- net 9: now reaches U5.15 (PB1)
- net 9: now also D8.2 (A), R11.1
- net PC2: now reaches U5.23 (PC0)
- net PC2: now also R3.2, R4.1
- new net: D3.2 (A), J2.2 (Pin_2)
- new net: D5.2 (A), J2.3 (Pin_3)
- new net: C2.1, D1.1 (K), D2.1 (K), R1.1, R7.1, U2.1 (VI)
- new net: C3.1, D3.1 (K), D5.1 (K), R3.1, R8.1, U3.1 (VI)
- new net: R11.2, U3.3 (VO)
- new net: Q3.2 (B), R15.2
- new net: C4.1, D4.1 (K), D6.1 (K), R5.1, R9.1, U4.1 (VI)
- new net: D12.2 (A), K3.A2, Q3.1 (C)
- new net: D6.2 (A), J3.3 (Pin_3)
- new net: D4.2 (A), J3.2 (Pin_2)
- new net RL3: J8.1 (Pin_1), K3.14
- no-connect marks 10 -> 17
